File: glove.kicad_sch (KiCad schematic)
At the start: 35 parts

Commit message: first commit
Parts:
- R?: value R_US -> 100k
Changed lines of the file:
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@@
       (effects (font (size 1.27 1.27)) (justify left))
     )
-    (property "Value" "R_US" (id 1) (at 96.52 78.74 90)
+    (property "Value" "100k" (id 1) (at 96.52 78.74 90)
       (effects (font (size 1.27 1.27)) (justify left))
     )
@@
     )
     (path "/9dd6204a-05e9-4976-a7d6-a404662245ff"
-      (reference "R?") (unit 1) (value "R_US") (footprint "")
+      (reference "R?") (unit 1) (value "100k") (footprint "")
     )
     (path "/0059bf36-c361-43a7-ae17-86e8b3787ce7"
